File: opencopcho.brd (EAGLE design)
At the start: 148 x 162 mm, 116 parts, among them CON1 PINHEAD_1X03-2.54, CON10 PINHEAD_1X03-2.54, CON11 PINHEAD_1X03-2.54, CON12 CON-4P-JST_GH-RA, CON13 CON-4P-JST_GH-RA, CON14 PINHEAD_1X02-2.54, CON15 CON-3P-3.81-RA, CON16 CON-3P-3.81-RA, CON17 CON-3P-3.81-RA, CON2 CON-3P-3.81-RA, CON3 CON-3P-3.81-RA, CON4 CON-3P-3.81-RA, CON5 CON-3P-3.81-RA, CON6 CON-3P-3.81-RA, CON7 CON_2P-3.5, CON8 CON-3P-3.81-RA, CON9 PINHEAD_1X03-2.54, IC1 TPS54260, IC3 ACS770, IC4 OPA342, IC5 VO3120-DIP8, IC6 MCP2542WFD, Q1 IRLML0030, Q2 IXFH120N30X3-STRAIGHT, Q3 IXFH120N30X3-STRAIGHT, Q4 IRLML0030, Q5 IXFH120N30X3-STRAIGHT, Q6 IXFH120N30X3-STRAIGHT, Q7 IXFH120N30X3-STRAIGHT, Q8 IXFH120N30X3-STRAIGHT, Q9 IXFH120N30X3-STRAIGHT, U1 LMV358

Commit message: some updates
Parts:
- removed BAR1: BUSBAR-150X10, zmey10:BUSBAR-150X10
- removed C17: (no value), rc:C0402
- removed C18, C19: 0.1u, rc:C0402
- removed C20, C21: 0.1u, rc:C0805
- removed C22, C23: DNM, rc:C0402
- removed CON10, CON11: PINHEAD_1X03-2.54, pinhead:1X03-PTH-2.54
- removed D10, D11, D12, D14, D18, D19, D20, D9: PESD3V3S1UB.115, TVS_diodes:SOD523
- removed D13, D15, D16: BAV99DW, Diodes:SOT363
- removed D17: B360B, Diodes:DO-214AA(SMB)
- removed HS1: HEATSINK-15X60X25, zmey10:HEATSINK_15X60X25
- removed IC3: ACS770, zmey10:CB-5-PFF
- removed IC4: OPA342, allegro:SOT23-5
- removed IC5: VO3120-DIP8, zmey10:DIL08
- removed IN+, IN-, OUT+, OUT-: PAD-7461383, PADS:7461383
- removed MODULE3: A0515S-2W, zmey10:B_S-2W
- removed MODULE4: NUCLEO-144-MORHO, zmey10:NUCLEO-144-MORPHO
- removed MODULE5: MCP2542_CLICK, zmey10:MCP2542_CLICK
- removed Q1, Q4: IRLML0030, mosfet:SOT23
- removed Q2, Q3, Q5, Q6, Q7, Q8, Q9: IXFH120N30X3-STRAIGHT, mosfet:TO247BV
- removed R10, R11: (no value), rc:R1206
- removed R12: (no value), rc:R0805
- removed R13, R15: 150K, rc:R0805
- removed R14: 2K, rc:R0805
- removed R16: 8K2, rc:R0805
- removed R17, R18, R37, R38: 6K8, rc:R0805
- removed R19, R20: 10K, rc:R0805
- removed R21, R22, R23, R24, R25, R26, R27, R28, R29, R30, R31, R32, R34, R35, R36: 33R, rc:R0805
- removed R33: 200R, rc:R0805
- removed R39: 000, rc:R0805
- removed U$1, U$2: CONNECTION, usb2can_master_lib:CONNECTION
- removed U1: LMV358, SparkFun-IC-Amplifiers:SO08
- added C1, C2: 0.1µF, C_digikey:C0603
- added CON18: PINHEAD_1X05-2.54-KEY, pinhead:1X05-PTH-2.54-KEY
- added D3: PMEG4020, Diodes:SOD123W
- added IC2: MCP2542WFD, serial_interfaces:SOIC8-3.9
- added MODULE1: NUCLEO-144-ZIO, stm32nucleo:NUCLEO-144-ZIO
- added R1, R3: 10R, rc:R0805
- added R2: 120R, rc:R0805
- added SJ3: (no value), usb2can_master_lib:RES_0
- CON1: value PINHEAD_1X03-2.54 -> (none); device pinhead:1X03-PTH-2.54 -> connect:D-09M
- CON15, CON16, CON17: value CON-3P-3.81-RA -> PINHEAD_1X05-2.54-KEY; device Connectors:DG381-3.81-03P -> pinhead:1X05-PTH-2.54-KEY
- CON2, CON4: value CON-3P-3.81-RA -> (none); device Connectors:DG381-3.81-03P -> connect:D-09F
- CON3: value CON-3P-3.81-RA -> (none); device Connectors:DG381-3.81-03P -> connect:D-09M
- CON5, CON6: value CON-3P-3.81-RA -> CON-4P-JST_GH-RA; device Connectors:DG381-3.81-03P -> Connectors:JST_GH-4P-RA
- CON7: value CON_2P-3.5 -> PINHEAD_1X02-2.54; device degson_connectors:3.5_RECEPTABLE_STRAIGHT_2P -> pinhead:1X02-PTH-2.54
- CON8: value CON-3P-3.81-RA -> PINHEAD_2X04-PLS; device Connectors:DG381-3.81-03P -> pinhead:2X04-PTH-2.54
- CON9: value PINHEAD_1X03-2.54 -> PINHEAD_2X04-PLS; device pinhead:1X03-PTH-2.54 -> pinhead:2X04-PTH-2.54
- D2: value PESD5V0S1BB,115 -> SM712; device TVS_diodes:SOD123 -> TVS_diodes:SOT23B-3
- D4, D6: value PESD5V0S1BB,115 -> SMBJ24CA-SMB; device TVS_diodes:SOD123 -> TVS_diodes:DO-214AA(SMB)
- D5, D7, D8: value PESD5V0S1BB,115 -> PMEG4020; device TVS_diodes:SOD123 -> Diodes:SOD123W
- R40: value 000 -> 120R
- moved D5 336.7 mm to (-33.0, -96.5)
- moved D4 332.7 mm to (-32.0, -107.0)
- moved CON4 306.6 mm to (-17.0, -26.5), turned to 180 degrees
- moved CON13 291.5 mm to (-15.0, -41.5), turned to 180 degrees
- moved D21 284.5 mm to (9.00, 5.00), turned to 180 degrees
- moved IC6 274.8 mm to (10.0, 23.0), turned to 180 degrees
- moved CON12 272.7 mm to (-5.00, -41.5), turned to 180 degrees
- moved D2 268.9 mm to (13.0, 5.00), turned to 180 degrees
- moved CON9 257.5 mm to (-23.0, 11.0), flipped to the bottom
- moved CON14 246.2 mm to (11.0, -35.0)
- moved CON7 244.5 mm to (-12.5, -35.0), turned to 180 degrees
- moved D8 243.2 mm to (-33.0, -104.0)
- moved D7 236.7 mm to (-33.0, -101.5)
- moved C13 228.7 mm to (-8.55, 22.6), turned to 270 degrees
- moved D6 227.3 mm to (-32.0, -93.5)
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Connections:
- net CAN_STBY renamed CAN1_STBY
- removed net !DUT_PWREN: Q4.1, R38.1
- removed net ADC1_INP15: MODULE4.CN12_37
- removed net ADC1_INP18: MODULE4.CN11_32
- removed net ADC1_INP19: MODULE4.CN12_11
- removed net ADC1_INP3: MODULE4.CN12_13
- removed net ADC3_INP10: MODULE4.CN11_38
- removed net ADC3_INP2: MODULE4.CN11_56
- removed net ADC3_INP3: MODULE4.CN11_11
- removed net ADC3_INP6: MODULE4.CN12_42
- removed net ADC3_INP7: MODULE4.CN11_54
- removed net ADC3_INP8: MODULE4.CN11_9
- removed net AIN1: D16.3, R29.2
- removed net AIN2: D16.6, R30.2
- removed net AIN3: D15.3, R31.2
- removed net AIN4: D15.6, R32.2
- removed net BRAKE_ON: Q1.1
- removed net CAN1_RX: IC6.4
- removed net CAN1_TX: IC6.1
- removed net CAN_RX: MODULE5.RX
- removed net CAN_TX: MODULE5.TX
- removed net CLICK_STBY: MODULE5.STB
- removed net CLOCK: D5.C, R21.2
- removed net CURRENT: IC3.3
- removed net DATA_CELL1: D8.C, R24.2
- removed net DATA_CELL2: D7.C, R23.2
- removed net DATA_CELL3: D6.C, R22.2
- removed net FDCAN1_RXFD: MODULE4.CN12_64
- removed net FDCAN1_TXFD: MODULE4.CN11_61
- removed net GATE: CON8.1, IC5.6, IC5.7
- removed net GPIO1: D12.C, R25.2
- removed net GPIO2: D11.C, R26.2
- removed net GPIO3: D10.C, R27.2
- removed net GPIO4: D9.C, R28.2
- removed net N$15: C17.2, D13.6, D14.C, IC4.3, R11.P$1, R12.2
- removed net N$17: R13.2, U1.6
- removed net N$18: C20.1, R14.2, U1.7
- removed net N$19: C20.2, R15.1, U1.2
- removed net N$20: CON1.3, R13.1, R14.1
- removed net N$21: R15.2, R16.1, R17.2, U1.3
- removed net N$22: R17.1, R18.1, U1.5
- removed net N$23: CON3.3, R21.1
- removed net N$24: CON3.2, R22.1
- removed net N$25: CON2.3, R24.1
- removed net N$26: CON3.1, R23.1
- removed net N$27: CON16.3, R25.1
- removed net N$28: CON15.1, R26.1
- removed net N$29: CON15.2, R27.1
- removed net N$30: CON15.3, R28.1
- removed net N$31: CON6.3, R29.1
- removed net N$32: CON5.1, R30.1
- removed net N$33: CON5.2, R31.1
- removed net N$34: CON5.3, R32.1
- removed net N$35: IC5.3, Q1.3
- removed net N$36: IC5.2, R33.2
- removed net N$37: CON7.1, D17.A
- removed net N$38: CON8.3, IC5.5, MODULE3.5
- removed net N$39: IC5.8, MODULE3.6
- removed net N$40: CON9.3, R34.1
- removed net N$41: CON10.3, R35.1
- removed net N$42: CON11.3, R36.1
- removed net N$43: HS1.P$1, HS1.P$2, HS1.P$3, HS1.P$4, HS1.P$5, OUT-.P$1, OUT-.P$10, OUT-.P$11, OUT-.P$12, OUT-.P$13, OUT-.P$14, OUT-.P$15, OUT-.P$16, OUT-.P$2, OUT-.P$3, OUT-.P$4, OUT-.P$5, OUT-.P$6, OUT-.P$7, OUT-.P$8, OUT-.P$9, Q2.D, Q3.D, Q5.D, Q6.D, Q7.D, Q8.D, Q9.D
- removed net N$44: BAR1.P$1, BAR1.P$2, BAR1.P$3, BAR1.P$4, BAR1.P$5, IN-.P$1, IN-.P$10, IN-.P$11, IN-.P$12, IN-.P$13, IN-.P$14, IN-.P$15, IN-.P$16, IN-.P$2, IN-.P$3, IN-.P$4, IN-.P$5, IN-.P$6, IN-.P$7, IN-.P$8, IN-.P$9, Q2.S, Q3.S, Q5.S, Q6.S, Q7.S, Q8.S, Q9.S, U$1.P$2
- removed net N$45: Q2.G, Q3.G, Q4.3, Q5.G, Q6.G, Q7.G, Q8.G, Q9.G, R37.1
- removed net N$46: CON12.1, CON13.1, R39.1
- removed net RCPWM1: D18.C, R34.2
- removed net RCPWM2: D19.C, R35.2
- removed net RCPWM3: D20.C, R36.2
- removed net TACHO: U1.1
- removed net TEMP1: C23.1, CON4.1, D2.C, R19.2
- removed net TEMP2: C22.1, CON4.2, D4.C, R20.2
- removed net TIM3_CH1: MODULE4.CN12_4
- removed net TIM3_CH2: MODULE4.CN12_19
- removed net TIM3_CH3: MODULE4.CN12_2
- removed net TIM3_CH4: MODULE4.CN12_1
- removed net USART2_CTS: MODULE4.CN11_40
- removed net USART2_RTS: MODULE4.CN11_39
- removed net USART2_RX: MODULE4.CN11_43
- removed net USART2_TX: MODULE4.CN11_41
- removed net VDC: IC3.CS1, IC3.CS3, IN+.P$1, IN+.P$10, IN+.P$11, IN+.P$12, IN+.P$13, IN+.P$14, IN+.P$15, IN+.P$16, IN+.P$2, IN+.P$3, IN+.P$4, IN+.P$5, IN+.P$6, IN+.P$7, IN+.P$8, IN+.P$9, R10.P$2
- removed net VOLTAGE: IC4.1, IC4.4
- new net CAN2_STBY: IC2.8
- new net N$3: CON12.1, CON13.1, D8.A
- new net N$5: CON7.2, R2.2
- new net N$6: C13.2, C14.2, L2.P$2, MODULE2.OUT+@1, MODULE2.OUT+@2, R8.2, SJ3.1
- new net N$8: CON5.1, CON6.1, D7.A
- net CAN_H: now also CON5.2, CON6.2, D2.1, IC2.7, R2.1
- net CAN_L: now also CON5.3, CON6.3, CON7.1, D2.2, IC2.6
- net FDCAN1_RX: now also IC6.4, MODULE1.CN7_4; no longer MODULE4.CN12_3
- net FDCAN1_TX: now also IC6.1, MODULE1.CN7_2; no longer MODULE4.CN12_5
- net FDCAN2_RX: now also IC2.4, MODULE1.CN7_7; no longer MODULE4.CN12_29
- net FDCAN2_TX: now also IC2.1, MODULE1.CN7_5; no longer MODULE4.CN12_17
- net GND: now also C1.P$2, C2.P$2, D2.3, IC2.2, MODULE1.CN8_11, MODULE1.CN8_13; no longer C17.1, C18.1, C19.2, C21.2, C22.2, C23.2, CON1.1, CON10.1, CON11.1, CON16.2, CON17.1, CON17.3, CON2.2, CON4.3, CON6.2, CON7.2, CON9.1, D10.A, D11.A, D12.A, D13.1, D14.A, D15.1, D15.4, D16.1, D16.4, D18.A, D19.A, D2.A, D20.A, D5.A, D7.A, D8.A, D9.A, IC3.2, IC4.2, MODULE3.2, MODULE4.CN11_19, MODULE4.CN11_20, MODULE4.CN11_22, MODULE4.CN11_49, MODULE4.CN11_60, MODULE4.CN11_71, MODULE4.CN11_72, MODULE4.CN11_8, MODULE4.CN12_20, MODULE4.CN12_39, MODULE4.CN12_54, MODULE4.CN12_63, MODULE4.CN12_71, MODULE4.CN12_72, MODULE4.CN12_9, MODULE5.GND@1, MODULE5.GND@2, Q1.2, Q4.2, R12.1, R18.2, U$1.P$1, U$2.P$1, U1.4
- net GNDD: now also CON5.4, CON5.M$0, CON5.M$1, CON6.4, CON6.M$0, CON6.M$1; no longer U$2.P$2
- net N$14: now also D5.A, D6.C, R3.1; no longer R10.P$1, R11.P$2
- net N$16: now also D3.A, D4.C, R1.1; no longer IC3.CS2, IC3.CS4, OUT+.P$1, OUT+.P$10, OUT+.P$11, OUT+.P$12, OUT+.P$13, OUT+.P$14, OUT+.P$15, OUT+.P$16, OUT+.P$2, OUT+.P$3, OUT+.P$4, OUT+.P$5, OUT+.P$6, OUT+.P$7, OUT+.P$8, OUT+.P$9
- net N$2: now also D3.C, D5.C; no longer D17.C
- net VDD_3V3: now also IC2.5; no longer D13.2, D15.2, D15.5, D16.2, D16.5, MODULE5.3V3, R38.2
- net VDD_5V: now also C1.P$1, C2.P$1, D7.C, D8.C, IC2.3, MODULE1.CN8_9, SJ3.2; no longer C13.2, C14.2, C18.2, C19.1, C21.1, CON1.2, CON10.2, CON11.2, CON16.1, CON17.2, CON2.1, CON6.1, CON9.2, IC3.1, IC4.5, L2.P$2, MODULE2.OUT+@1, MODULE2.OUT+@2, MODULE3.1, MODULE5.5V, R16.2, R19.1, R20.1, R33.1, R37.2, R39.2, R8.2, U1.8
Routing:
- net VDD_5V: track 9.55 -> 0.00 mm
- net N$6: track 0.00 -> 9.55 mm
- removed copper zone on layer 1, net N$16
- removed copper zone on layer 16, net N$16
- removed copper zone on layer 1, net N$43
- removed copper zone on layer 16, net N$43
- removed copper zone on layer 1, net N$44
- removed copper zone on layer 16, net N$44
- removed copper zone on layer 1, net VDC
- removed copper zone on layer 16, net VDC
Other:
- board outline removed

Commit message: updates
Parts:
- removed CON17, CON18: PINHEAD_1X05-2.54-KEY, pinhead:1X05-PTH-2.54-KEY
- added CON10, CON11: PINHEAD_1X05-2.54-KEY, pinhead:1X05-PTH-2.54-KEY
- moved CON15 4.00 mm to (-7.00, -2.50)
- moved CON16 4.00 mm to (-21.0, -2.50)
- moved SJ3 0.95 mm to (-2.95, 27.0), turned to 90 degrees
- moved CON9 0.25 mm to (-22.9, 10.8)
- moved CON8 0.17 mm to (22.9, 30.1)
Connections:
- net N$2 renamed VDD_24V
- removed net CAN_H: CON12.2, CON13.2, CON5.2, CON6.2, D2.1, D21.1, IC2.7, IC6.7, R2.1, R40.1
- removed net CAN_L: CON12.3, CON13.3, CON14.1, CON5.3, CON6.3, CON7.1, D2.2, D21.2, IC2.6, IC6.6
- new net CAN1_H: CON1.7, CON15.4, CON16.4, CON2.7, CON5.2, CON6.2, D2.1, IC2.7, R2.1
- new net CAN1_L: CON1.2, CON15.3, CON16.3, CON2.2, CON5.3, CON6.3, CON7.1, D2.2, IC2.6
- new net CAN1_SHIELD: CON15.2, CON16.2, CON2.5
- new net CAN1_VDD: CON1.9, CON15.5, CON16.5, CON2.9, R3.2
- new net CAN2_H: CON10.4, CON11.4, CON12.2, CON13.2, CON3.7, CON4.7, D21.1, IC6.7, R40.1
- new net CAN2_L: CON10.3, CON11.3, CON12.3, CON13.3, CON14.1, CON3.2, CON4.2, D21.2, IC6.6
- new net CAN2_SHIELD: CON10.2, CON11.2, CON3.5
- new net CAN2_VDD: CON10.5, CON11.5, CON3.9, R1.2
- net GND: now also CON1.6, CON10.1, CON11.1, CON15.1, CON16.1, CON2.6, CON3.6, CON4.6
Routing:
- added copper zone on layer 1, net N$6
- removed copper zone on layer 1, net VDD_5V

Commit message: updates
Parts:
- removed CON8, CON9: PINHEAD_2X04-PLS, pinhead:2X04-PTH-2.54
- removed MODULE1: NUCLEO-144-ZIO, stm32nucleo:NUCLEO-144-ZIO
- added CON17: PINHEAD_2X17-TH-FEMALE-LONG, pinhead:2X17-PTH-2.54-FEMALE-LONG_PINS
- added CON18: PINHEAD_2X15-2.54-FEMALE-LONG, pinhead:2X15-PTH-2.54-FEMALE-LONG-PINS
- added CON19: PINHEAD_2X08-TH-FEMALE-LONG, pinhead:2X08-PTH-2.54-FEMALE-LONG-PINS
- added CON20: PINHEAD_2X10-2.54-TH-FEMALE-LONG, pinhead:2X10-PTH-2.54-FEMALE-LONG-PINS
- added D9: SMBJ5.0CA-SMB, TVS_diodes:DO-214AA(SMB)
- added LED1, LED2: LED-0805, rc:LED0805
- added R10, R4: 470R, rc:R0805
- CON1, CON3: device connect:D-09M -> Connectors:D-09M
- CON2, CON4: device connect:D-09F -> Connectors:D-09M
- D1: value B360B-SMB -> B360B; device eth_conv_master_lib:SMB -> Diodes:DO-214AA(SMB)
- IC1: device eth_conv_master_lib:MSOP10 -> dc-dc:MSOP10
- L2: value 4.7uH -> 22µH; device eth_conv_master_lib:SWPA6045S3R3N -> power_inductors:SRP6540
- MODULE2: value GW1584 -> GW1584_MODULE; device ali_modules:GW1584 -> dc-dc:GW1584_MODULE
- moved R1 137.5 mm to (-6.35, 22.4)
- moved D3 133.7 mm to (-17.6, 22.9), turned to 180 degrees
- moved D4 129.7 mm to (-13.6, 21.4), turned to 270 degrees
- moved R3 122.3 mm to (-6.35, 20.4)
- moved D5 117.7 mm to (-17.6, 20.2), turned to 180 degrees
- moved D6 117.0 mm to (-10.1, 21.4), turned to 270 degrees
- moved D8 75.5 mm to (0.00, -36.0)
- moved D7 71.0 mm to (0.00, -38.6)
- moved CON11 38.6 mm to (-15.5, -15.0), turned to 270 degrees
- moved CON16 38.0 mm to (17.0, -1.50), turned to 270 degrees
- moved CON7 36.2 mm to (22.8, -43.0), turned to 0 degrees
- moved CON10 34.8 mm to (-15.5, -29.0), turned to 270 degrees
- moved CON14 34.4 mm to (-22.5, -43.0), turned to 180 degrees
- moved R2 33.0 mm to (15.4, -37.0)
- moved R40 31.8 mm to (-15.8, -37.0)
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Connections:
- removed net FDCAN1_RX: IC6.4, MODULE1.CN7_4
- removed net FDCAN1_TX: IC6.1, MODULE1.CN7_2
- removed net FDCAN2_RX: IC2.4, MODULE1.CN7_7
- removed net FDCAN2_TX: IC2.1, MODULE1.CN7_5
- removed net GNDD: CON12.4, CON12.M$0, CON12.M$1, CON13.4, CON13.M$0, CON13.M$1, CON5.4, CON5.M$0, CON5.M$1, CON6.4, CON6.M$0, CON6.M$1
- new net N$2: LED1.A, R4.1
- new net N$7: LED2.A, R10.1
- new net PB12/FDCAN1_RX: CON20.7, IC6.4
- new net PB13/FDCAN1_TX: CON20.5, IC6.1
- new net PB15/CAN2_LED: CON20.3, R10.2
- new net PC6/CAN1_LED: CON20.1, R4.2
- new net PD0/FDCAN2_RX: CON18.25, IC2.4
- new net PD1/FDCAN2_TX: CON18.27, IC2.1
- net AA1: now also L2.1; no longer L2.P$1
- net CAN1_SHIELD: now also CON1.5
- net CAN2_SHIELD: now also CON4.5
- net CAN2_VDD: now also CON4.9
- net GND: now also CON12.4, CON12.M$0, CON12.M$1, CON13.4, CON13.M$0, CON13.M$1, CON19.11, CON19.13, CON5.4, CON5.M$0, CON5.M$1, CON6.4, CON6.M$0, CON6.M$1, D9.C, LED1.C, LED2.C; no longer MODULE1.CN8_11, MODULE1.CN8_13
- net N$6: now also L2.2; no longer L2.P$2
- net VDD_5V: now also CON19.9, D9.A; no longer MODULE1.CN8_9
Routing:
- net CAN2_L: track 0.00 -> 153.9 mm
- net VDD_5V: track 0.00 -> 153.6 mm, vias 0 -> 1
- net CAN1_L: track 0.00 -> 144.5 mm
- net CAN2_H: track 0.00 -> 137.0 mm
- net CAN1_H: track 0.00 -> 136.3 mm
- net PD1/FDCAN2_TX: track 0.00 -> 98.7 mm, vias 0 -> 2
- net PD0/FDCAN2_RX: track 0.00 -> 92.1 mm, vias 0 -> 2
- net CAN2_VDD: track 0.00 -> 91.2 mm
- net CAN1_VDD: track 0.00 -> 82.3 mm
- net CAN2_SHIELD: track 0.00 -> 57.6 mm
- net CAN1_SHIELD: track 0.00 -> 57.1 mm
- net N$3: track 0.00 -> 22.8 mm, vias 0 -> 4
- net N$8: track 0.00 -> 17.7 mm
- net PB12/FDCAN1_RX: track 0.00 -> 16.1 mm
- net PB15/CAN2_LED: track 0.00 -> 12.8 mm
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- added copper zone on layer 16, net GND
- added copper zone on layer 1, net VDD_24V
- removed copper zone on layer 1, net N$13
- removed copper zone on layer 1, net VBAT
Other:
- board outline added: 51 x 87.5 mm
- board text added: "CAN1"
- board text added: "CAN2"

Commit message: opencopcho is basically done
Parts:
- added U$1: (no value), pixhawk_esc_1.5_master_lib:ZUBAX_LOGO_5X10
- added U$4: (no value), logo:OSHW-10.5X11.5
- moved R1 1.50 mm to (-4.85, 22.4)
- moved R3 1.50 mm to (-4.85, 20.4)
- moved D6 1.00 mm to (-9.05, 21.4)
- moved D4 0.50 mm to (-13.1, 21.4)
Connections:
- removed net CAN1_STBY: IC6.8
- removed net CAN2_STBY: IC2.8
- net VDD_3V3: now also CON19.7
Routing:
- net VDD_3V3: track 0.00 -> 57.8 mm, vias 0 -> 2
- net CAN2_SHIELD: track 57.6 -> 44.7 mm
- net PD1/FDCAN2_TX: track 98.7 -> 90.1 mm
- net CAN2_L: track 153.9 -> 151.3 mm
- net CAN2_H: track 137.0 -> 135.2 mm
- net N$14: track 12.0 -> 13.5 mm
- net CAN1_L: track 144.5 -> 143.1 mm
- net N$16: track 12.2 -> 13.4 mm
- net CAN1_VDD: track 82.3 -> 82.9 mm
- net CAN2_VDD: track 91.2 -> 91.8 mm
- net CAN1_H: track 136.3 -> 135.7 mm
- net GND: vias 28 -> 30
Other:
- board text added: "Opencopcho V0.1"

Commit message: fiducials
Parts:
- added U$11, U$5, U$6, U$7: FIDUCIALMOUNT, usb2can_master_lib:FIDUCIA-MOUNT
Routing:
- net GND: vias 30 -> 74

Commit message: temporary  BOM link
Routing:
- net GND: vias 74 -> 91
Changed lines of the file:
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@@
 <drawing>
 <settings>
-<setting alwaysvectorfont="no"/>
+<setting alwaysvectorfont="yes"/>
 <setting verticaltext="up"/>
 </settings>
@@
 <layer number="14" name="Route14" color="22" fill="1" visible="no" active="no"/>
 <layer number="15" name="Route15" color="23" fill="1" visible="no" active="no"/>
-<layer number="16" name="Bottom" color="1" fill="1" visible="yes" active="yes"/>
+<layer number="16" name="Bottom" color="1" fill="1" visible="no" active="yes"/>
 <layer number="17" name="Pads" color="2" fill="1" visible="yes" active="yes"/>
 <layer number="18" name="Vias" color="2" fill="1" visible="yes" active="yes"/>
@@
 <text x="19.15" y="39" size="1.5" layer="21" font="vector" ratio="15" align="center">CAN2</text>
 <text x="-7.45" y="40.75" size="1.45" layer="16" font="vector" ratio="15" rot="MR0" align="center">Opencopcho V0.1</text>
+<rectangle x1="-7.8" y1="37.15" x2="-6.5" y2="38.35" layer="22"/>
+<rectangle x1="-3.05" y1="32.55" x2="-1.85" y2="33.75" layer="22"/>
+<rectangle x1="-12.45" y1="32.5" x2="-11.2" y2="33.8" layer="22"/>
+<rectangle x1="-10.9" y1="29.25" x2="-9.9" y2="30.55" layer="22"/>
+<rectangle x1="-4.35" y1="29.25" x2="-3.4" y2="30.6" layer="22"/>
+<rectangle x1="-11" y1="35.75" x2="-9.85" y2="37" layer="22"/>
 </plain>
 <attributes>
@@
 <via x="-20.1" y="21.55" extent="1-16" drill="0.5" diameter="1"/>
 <via x="-19.45" y="41" extent="1-16" drill="0.5" diameter="1"/>
+<via x="20.05" y="32.7" extent="1-16" drill="0.5" diameter="1"/>
+<via x="15.35" y="38.5" extent="1-16" drill="0.5" diameter="1"/>
+<via x="23.35" y="36.25" extent="1-16" drill="0.5" diameter="1"/>
+<via x="23.55" y="41.05" extent="1-16" drill="0.5" diameter="1"/>
+<via x="5.7" y="40.85" extent="1-16" drill="0.5" diameter="1"/>
+<via x="4.5" y="32.1" extent="1-16" drill="0.5" diameter="1"/>
+<via x="4.4" y="34.9" extent="1-16" drill="0.5" diameter="1"/>
+<via x="1.1" y="35.5" extent="1-16" drill="0.5" diameter="1"/>
+<via x="1.2" y="33" extent="1-16" drill="0.5" diameter="1"/>
+<via x="-13.25" y="33.75" extent="1-16" drill="0.5" diameter="1"/>
+<via x="-11.2" y="37.35" extent="1-16" drill="0.5" diameter="1"/>
+<via x="-14" y="37.35" extent="1-16" drill="0.5" diameter="1"/>
+<via x="-19.05" y="35.65" extent="1-16" drill="0.5" diameter="1"/>
+<via x="-19.2" y="33.95" extent="1-16" drill="0.5" diameter="1"/>
+<via x="-19.1" y="32" extent="1-16" drill="0.5" diameter="1"/>
+<via x="-15.05" y="25.9" extent="1-16" drill="0.5" diameter="1"/>
+<via x="-11.2" y="34.15" extent="1-16" drill="0.5" diameter="1"/>
 </signal>
 <signal name="N$10">

Commit message: silk updates
Parts:
- added R11, R12: (no value), rc:R1206
- added SJ1, SJ2: (no value), usb2can_master_lib:RES_0
Connections:
- net CAN1_SHIELD: now also R11.P$1, SJ2.1
- net CAN2_SHIELD: now also R12.P$1, SJ1.1
- net GND: now also R11.P$2, R12.P$2, SJ1.2, SJ2.2
Routing:
- net CAN2_SHIELD: track 44.7 -> 46.3 mm
- net CAN1_SHIELD: track 57.1 -> 57.8 mm
Other:
- board text added: "24V"
- board text added: "CANH"
- board text added: "CANL"
- board text added: "CAN_H"
- board text added: "CAN_L"
- board text added: "GND"
- board text added: "SHIELD"
