File: opencopcho.sch (EAGLE design)
At the start: 116 parts, among them CON1 PINHEAD_1X03-2.54, CON10 PINHEAD_1X03-2.54, CON11 PINHEAD_1X03-2.54, CON12 CON-4P-JST_GH-RA, CON13 CON-4P-JST_GH-RA, CON14 PINHEAD_1X02-2.54, CON15 CON-3P-3.81-RA, CON16 CON-3P-3.81-RA, CON17 CON-3P-3.81-RA, CON2 CON-3P-3.81-RA, CON3 CON-3P-3.81-RA, CON4 CON-3P-3.81-RA, CON5 CON-3P-3.81-RA, CON6 CON-3P-3.81-RA, CON7 CON_2P-3.5, CON8 CON-3P-3.81-RA, CON9 PINHEAD_1X03-2.54, IC1 TPS54260, IC3 ACS770, IC4 OPA342, IC5 VO3120-DIP8, IC6 MCP2542WFD, Q1 IRLML0030, Q2 IXFH120N30X3-STRAIGHT, Q3 IXFH120N30X3-STRAIGHT, Q4 IRLML0030, Q5 IXFH120N30X3-STRAIGHT, Q6 IXFH120N30X3-STRAIGHT, Q7 IXFH120N30X3-STRAIGHT, Q8 IXFH120N30X3-STRAIGHT, Q9 IXFH120N30X3-STRAIGHT, U1 LMV358

Commit message: some updates
Parts:
- removed BAR1: BUSBAR-150X10, zmey10:BUSBAR-150X10
- removed C17: (no value), rc:C-0402
- removed C18, C19: 0.1u, rc:C-0402
- removed C20, C21: 0.1u, rc:C-0805
- removed C22, C23: DNM, rc:C-0402
- removed CON10, CON11: PINHEAD_1X03-2.54, pinhead:PINHEAD_1X03-2.54
- removed D10, D11, D12, D14, D18, D19, D20, D9: PESD3V3S1UB.115, TVS_diodes:PESD3V3S1UB.115
- removed D13, D15, D16: BAV99DW, Diodes:BAV99DW
- removed D17: B360B, Diodes:B360B
- removed HS1: HEATSINK-15X60X25, zmey10:HEATSINK-15X60X25
- removed IC3: ACS770, zmey10:ACS770
- removed IC4: OPA342, allegro:OPA342
- removed IC5: VO3120-DIP8, zmey10:VO3120-DIP8
- removed IN+, IN-, OUT+, OUT-: PAD-7461383, PADS:PAD-7461383
- removed MODULE3: A0515S-2W, zmey10:A0515S-2W
- removed MODULE4: NUCLEO-144-MORHO, zmey10:NUCLEO-144-MORHO
- removed MODULE5: MCP2542_CLICK, zmey10:MCP2542_CLICK
- removed Q1, Q4: IRLML0030, mosfet:IRLML0030
- removed Q2, Q3, Q5, Q6, Q7, Q8, Q9: IXFH120N30X3-STRAIGHT, mosfet:IXFH120N30X3-STRAIGHT
- removed R10, R11: (no value), rc:R-1206
- removed R12: (no value), rc:R-0805
- removed R13, R15: 150K, rc:R-0805
- removed R14: 2K, rc:R-0805
- removed R16: 8K2, rc:R-0805
- removed R17, R18, R37, R38: 6K8, rc:R-0805
- removed R19, R20: 10K, rc:R-0805
- removed R21, R22, R23, R24, R25, R26, R27, R28, R29, R30, R31, R32, R34, R35, R36: 33R, rc:R-0805
- removed R33: 200R, rc:R-0805
- removed R39: 000, rc:R-0805
- removed U$1, U$2: CONNECTION, usb2can_master_lib:CONNECTION
- removed U1: LMV358, SparkFun-IC-Amplifiers:LMV358SOIC
- added C1, C2: 0.1µF, C_digikey:0.1µF-16V_10%_X7R-0603
- added CON18: PINHEAD_1X05-2.54-KEY, pinhead:PINHEAD_1X05-2.54-KEY
- added D3: PMEG4020, Diodes:PMEG4020
- added IC2: MCP2542WFD, serial_interfaces:MCP2542WFD
- added MODULE1: NUCLEO-144-ZIO, stm32nucleo:NUCLEO-144-ZIO
- added R1, R3: 10R, rc:R-5%-0805
- added R2: 120R, rc:R-1%-0805
- added SJ3: (no value), usb2can_master_lib:SOLDER_JOINT
- CON1: value PINHEAD_1X03-2.54 -> (none); device pinhead:PINHEAD_1X03-2.54 -> connect:DB9M
- CON15, CON16, CON17: value CON-3P-3.81-RA -> PINHEAD_1X05-2.54-KEY; device Connectors:CON-3P-3.81-RA -> pinhead:PINHEAD_1X05-2.54-KEY
- CON2, CON4: value CON-3P-3.81-RA -> (none); device Connectors:CON-3P-3.81-RA -> connect:DB9F
- CON3: value CON-3P-3.81-RA -> (none); device Connectors:CON-3P-3.81-RA -> connect:DB9M
- CON5, CON6: value CON-3P-3.81-RA -> CON-4P-JST_GH-RA; device Connectors:CON-3P-3.81-RA -> Connectors:CON-4P-JST_GH-RA
- CON7: value CON_2P-3.5 -> PINHEAD_1X02-2.54; device degson_connectors:CON_2P-3.5 -> pinhead:PINHEAD_1X02-2.54
- CON8: value CON-3P-3.81-RA -> PINHEAD_2X04-PLS; device Connectors:CON-3P-3.81-RA -> pinhead:PINHEAD_2X04-PLS
- CON9: value PINHEAD_1X03-2.54 -> PINHEAD_2X04-PLS; device pinhead:PINHEAD_1X03-2.54 -> pinhead:PINHEAD_2X04-PLS
- D2: value PESD5V0S1BB,115 -> SM712; device TVS_diodes:PESD5V0S1BB,115 -> TVS_diodes:SM712
- D4, D6: value PESD5V0S1BB,115 -> SMBJ24CA-SMB; device TVS_diodes:PESD5V0S1BB,115 -> TVS_diodes:SMBJ24CA-SMB
- D5, D7, D8: value PESD5V0S1BB,115 -> PMEG4020; device TVS_diodes:PESD5V0S1BB,115 -> Diodes:PMEG4020
- R40: value 000 -> 120R; device rc:R-0805 -> rc:R-1%-0805
Connections:
- net CAN_STBY renamed CAN1_STBY
- removed net !DUT_PWREN: Q4.G, R38.1
- removed net ADC1_INP15: MODULE4CN12.PA3
- removed net ADC1_INP18: MODULE4CN11.PA4
- removed net ADC1_INP19: MODULE4CN12.PA5
- removed net ADC1_INP3: MODULE4CN12.PA6
- removed net ADC3_INP10: MODULE4CN11.PC0
- removed net ADC3_INP2: MODULE4CN11.PF9
- removed net ADC3_INP3: MODULE4CN11.PF7
- removed net ADC3_INP6: MODULE4CN12.PF10
- removed net ADC3_INP7: MODULE4CN11.PF8
- removed net ADC3_INP8: MODULE4CN11.PF6
- removed net AIN1: D16D2.COMMON, R29.2
- removed net AIN2: D16D1.COMMON, R30.2
- removed net AIN3: D15D2.COMMON, R31.2
- removed net AIN4: D15D1.COMMON, R32.2
- removed net BRAKE_ON: Q1.G
- removed net CAN1_RX: IC6.RXD
- removed net CAN1_TX: IC6.TXD
- removed net CAN_RX: MODULE5.RX
- removed net CAN_TX: MODULE5.TX
- removed net CLICK_STBY: MODULE5.STBY
- removed net CLOCK: D5.C, R21.2
- removed net CURRENT: IC3.VOUT
- removed net DATA_CELL1: D8.C, R24.2
- removed net DATA_CELL2: D7.C, R23.2
- removed net DATA_CELL3: D6.C, R22.2
- removed net FDCAN1_RXFD: MODULE4CN12.PE0
- removed net FDCAN1_TXFD: MODULE4CN11.PE1
- removed net GATE: CON8.1, IC5.VO@1, IC5.VO@2
- removed net GPIO1: D12.C, R25.2
- removed net GPIO2: D11.C, R26.2
- removed net GPIO3: D10.C, R27.2
- removed net GPIO4: D9.C, R28.2
- removed net N$15: C17.2, D13D1.COMMON, D14.C, IC4.+, R11.1, R12.2
- removed net N$17: R13.2, U1G2.-IN
- removed net N$18: C20.1, R14.2, U1G2.OUT
- removed net N$19: C20.2, R15.1, U1G1.-IN
- removed net N$20: CON1.3, R13.1, R14.1
- removed net N$21: R15.2, R16.1, R17.2, U1G1.+IN
- removed net N$22: R17.1, R18.1, U1G2.+IN
- removed net N$23: CON3.3, R21.1
- removed net N$24: CON3.2, R22.1
- removed net N$25: CON2.3, R24.1
- removed net N$26: CON3.1, R23.1
- removed net N$27: CON16.3, R25.1
- removed net N$28: CON15.1, R26.1
- removed net N$29: CON15.2, R27.1
- removed net N$30: CON15.3, R28.1
- removed net N$31: CON6.3, R29.1
- removed net N$32: CON5.1, R30.1
- removed net N$33: CON5.2, R31.1
- removed net N$34: CON5.3, R32.1
- removed net N$35: IC5.C, Q1.D
- removed net N$36: IC5.A, R33.2
- removed net N$37: CON7.1, D17.A
- removed net N$38: CON8.3, IC5.VEE, MODULE3.0V
- removed net N$39: IC5.VCC, MODULE3.VO+
- removed net N$40: CON9.3, R34.1
- removed net N$41: CON10.3, R35.1
- removed net N$42: CON11.3, R36.1
- removed net N$43: HS1.P$1, OUT-.P$1, Q2.D, Q3.D, Q5.D, Q6.D, Q7.D, Q8.D, Q9.D
- removed net N$44: BAR1.P$1, IN-.P$1, Q2.S, Q3.S, Q5.S, Q6.S, Q7.S, Q8.S, Q9.S, U$1.P$2
- removed net N$45: Q2.G, Q3.G, Q4.D, Q5.G, Q6.G, Q7.G, Q8.G, Q9.G, R37.1
- removed net N$46: CON12.1, CON13.1, R39.1
- removed net RCPWM1: D18.C, R34.2
- removed net RCPWM2: D19.C, R35.2
- removed net RCPWM3: D20.C, R36.2
- removed net TACHO: U1G1.OUT
- removed net TEMP1: C23.1, CON4.1, D2.C, R19.2
- removed net TEMP2: C22.1, CON4.2, D4.C, R20.2
- removed net TIM3_CH1: MODULE4CN12.PC6
- removed net TIM3_CH2: MODULE4CN12.PC7
- removed net TIM3_CH3: MODULE4CN12.PC8
- removed net TIM3_CH4: MODULE4CN12.PC9
- removed net USART2_CTS: MODULE4CN11.PD3
- removed net USART2_RTS: MODULE4CN11.PD4
- removed net USART2_RX: MODULE4CN11.PD6
- removed net USART2_TX: MODULE4CN11.PD5
- removed net VDC: IC3.CS1, IN+.P$1, R10.2
- removed net VOLTAGE: IC4.-, IC4.OUT
- new net CAN2_STBY: IC2.STBY
- new net N$3: CON12.1, CON13.1, D8.A
- new net N$5: CON7.2, R2.2
- new net N$6: C13.2, C14.2, L2.P$2, MODULE2.OUT+, R8.2, SJ3.1
- new net N$8: CON5.1, CON6.1, D7.A
- net CAN_H: now also CON5.2, CON6.2, D2.C3, IC2.CANH, R2.1
- net CAN_L: now also CON5.3, CON6.3, CON7.1, D2.C2, IC2.CANL
- net FDCAN1_RX: now also IC6.RXD, MODULE1CN7.PB9/D14; no longer MODULE4CN12.PB8
- net FDCAN1_TX: now also IC6.TXD, MODULE1CN7.PB8/D15; no longer MODULE4CN12.PB9
- net FDCAN2_RX: now also IC2.RXD, MODULE1CN7.PB12; no longer MODULE4CN12.PB5
- net FDCAN2_TX: now also IC2.TXD, MODULE1CN7.PB13; no longer MODULE4CN12.PB6
- net GND: now also C1.2, C2.2, D2.P$1, IC2.GND, MODULE1CN8.GND@1, MODULE1CN8.GND@2; no longer C17.1, C18.1, C19.2, C21.2, C22.2, C23.2, CON1.1, CON10.1, CON11.1, CON16.2, CON17.1, CON17.3, CON2.2, CON4.3, CON6.2, CON7.2, CON9.1, D10.A, D11.A, D12.A, D13D1.A, D14.A, D15D1.A, D15D2.A, D16D1.A, D16D2.A, D18.A, D19.A, D2.A, D20.A, D5.A, D7.A, D8.A, D9.A, IC3.GND, IC4.V-, MODULE3.GND, MODULE4CN11.GND@1, MODULE4CN11.GND@2, MODULE4CN11.GND@3, MODULE4CN11.GND@4, MODULE4CN11.GND@5, MODULE4CN11.GND@6, MODULE4CN11.GND@7, MODULE4CN11.GND@8, MODULE4CN12.GND@1, MODULE4CN12.GND@2, MODULE4CN12.GND@3, MODULE4CN12.GND@4, MODULE4CN12.GND@5, MODULE4CN12.GND@6, MODULE4CN12.GND@7, MODULE5.GND, Q1.S, Q4.S, R12.1, R18.2, U$1.P$1, U$2.P$1, U1G3.P$V-
- net GNDD: now also CON5.4, CON5.GND, CON6.4, CON6.GND; no longer U$2.P$2
- net N$14: now also D5.A, D6.C, R3.1; no longer R10.1, R11.2
- net N$16: now also D3.A, D4.C, R1.1; no longer IC3.CS2, OUT+.P$1
- net N$2: now also D3.C, D5.C; no longer D17.C
- net VDD_3V3: now also IC2.VIO; no longer D13D1.C, D15D1.C, D15D2.C, D16D1.C, D16D2.C, MODULE5.3V3, R38.2
- net VDD_5V: now also C1.1, C2.1, D7.C, D8.C, IC2.VCC, MODULE1CN8.5V, SJ3.2; no longer C13.2, C14.2, C18.2, C19.1, C21.1, CON1.2, CON10.2, CON11.2, CON16.1, CON17.2, CON2.1, CON6.1, CON9.2, IC3.VCC, IC4.V+, L2.P$2, MODULE2.OUT+, MODULE3.VIN, MODULE5.5V, R16.2, R19.1, R20.1, R33.1, R37.2, R39.2, R8.2, U1G3.P$V+
Other:
- note removed: "AVOID USING"
- note removed: "Battery negative"
- note removed: "Battery positive"
- note removed: "Brake resistor control"
- note removed: "Current sensing"
- note removed: "DUT negative"
- note removed: "DUT positive"
- note removed: "For connection of load cells with HX711 acqusition board"
- note removed: "GPIO"
- note removed: "GPIO SET"
- note removed: "JUST IN CASE ANALOG INPUTS"
- note removed: "JUST IN CASE GPIO"
- note removed: "Just in case RCPWM"
- note removed: "Optical tachometer"
- note removed: "Pull DUT_PWREN low to enable power for DUT"
- note removed: "TIMER"
- note removed: "Thermistor connection"
- note removed: "UART"
- note removed: "Voltage sensing"
- moved on the sheet: C10, C11, C12, C13, C14, C15, C16, C8, CON14, CON5, CON6, D1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

Commit message: updates
Parts:
- renumbered CON17 to CON10, CON18 to CON11
Connections:
- net N$2 renamed VDD_24V
- removed net CAN_H: CON12.2, CON13.2, CON5.2, CON6.2, D2.C3, D21.C3, IC2.CANH, IC6.CANH, R2.1, R40.1
- removed net CAN_L: CON12.3, CON13.3, CON14.1, CON5.3, CON6.3, CON7.1, D2.C2, D21.C2, IC2.CANL, IC6.CANL
- new net CAN1_H: CON1.7, CON15.4, CON16.4, CON2.7, CON5.2, CON6.2, D2.C3, IC2.CANH, R2.1
- new net CAN1_L: CON1.2, CON15.3, CON16.3, CON2.2, CON5.3, CON6.3, CON7.1, D2.C2, IC2.CANL
- new net CAN1_SHIELD: CON15.2, CON16.2, CON2.5
- new net CAN1_VDD: CON1.9, CON15.5, CON16.5, CON2.9, R3.2
- new net CAN2_H: CON10.4, CON11.4, CON12.2, CON13.2, CON3.7, CON4.7, D21.C3, IC6.CANH, R40.1
- new net CAN2_L: CON10.3, CON11.3, CON12.3, CON13.3, CON14.1, CON3.2, CON4.2, D21.C2, IC6.CANL
- new net CAN2_SHIELD: CON10.2, CON11.2, CON3.5
- new net CAN2_VDD: CON10.5, CON11.5, CON3.9, R1.2
- net GND: now also CON1.6, CON10.1, CON11.1, CON15.1, CON16.1, CON2.6, CON3.6, CON4.6
Other:
- moved on the sheet: CON8, CON9, D3, D4, D5, D6, R1, R3

Commit message: updates
Parts:
- removed CON8, CON9: PINHEAD_2X04-PLS, pinhead:PINHEAD_2X04-PLS
- removed MODULE1: NUCLEO-144-ZIO, stm32nucleo:NUCLEO-144-ZIO
- added CON17: PINHEAD_2X17-TH-FEMALE-LONG, pinhead:PINHEAD_2X17-TH-FEMALE-LONG
- added CON18: PINHEAD_2X15-2.54-FEMALE-LONG, pinhead:PINHEAD_2X15-2.54-FEMALE-LONG
- added CON19: PINHEAD_2X08-TH-FEMALE-LONG, pinhead:PINHEAD_2X08-TH-FEMALE-LONG
- added CON20: PINHEAD_2X10-2.54-TH-FEMALE-LONG, pinhead:PINHEAD_2X10-2.54-TH-FEMALE-LONG
- added D9: SMBJ5.0CA-SMB, TVS_diodes:SMBJ5.0CA-SMB
- added LED1, LED2: LED-0805, rc:LED-0805
- added R10, R4: 470R, rc:R-5%-0805
- C16: device C_digikey:33P-50V_5%_NP0-0603 -> C_digikey:33PF-50V_5%_NP0-0603
- CON1, CON3: device connect:DB9M -> Connectors:DB9-M
- CON2, CON4: device connect:DB9F -> Connectors:DB9-M
- D1: value B360B-SMB -> B360B; device eth_conv_master_lib:B360B-SMB -> Diodes:B360B
- IC1: device eth_conv_master_lib:TPS54260 -> dc-dc:TPS54260
- L2: value 4.7uH -> 22µH; device eth_conv_master_lib:L -> power_inductors:22µH-22U-SRP6540
- MODULE2: value GW1584 -> GW1584_MODULE; device ali_modules:GW1584 -> dc-dc:GW1584_MODULE
- R8: device rc:R-0603 -> rc:R-1%-0603
Connections:
- removed net FDCAN1_RX: IC6.RXD, MODULE1CN7.PB9/D14
- removed net FDCAN1_TX: IC6.TXD, MODULE1CN7.PB8/D15
- removed net FDCAN2_RX: IC2.RXD, MODULE1CN7.PB12
- removed net FDCAN2_TX: IC2.TXD, MODULE1CN7.PB13
- removed net GNDD: CON12.4, CON12.GND, CON13.4, CON13.GND, CON5.4, CON5.GND, CON6.4, CON6.GND
- new net N$2: LED1.A, R4.1
- new net N$7: LED2.A, R10.1
- new net PB12/FDCAN1_RX: CON20.7, IC6.RXD
- new net PB13/FDCAN1_TX: CON20.5, IC6.TXD
- new net PB15/CAN2_LED: CON20.3, R10.2
- new net PC6/CAN1_LED: CON20.1, R4.2
- new net PD0/FDCAN2_RX: CON18.25, IC2.RXD
- new net PD1/FDCAN2_TX: CON18.27, IC2.TXD
- net CAN1_SHIELD: now also CON1.5
- net CAN2_SHIELD: now also CON4.5
- net CAN2_VDD: now also CON4.9
- net GND: now also CON12.4, CON12.GND, CON13.4, CON13.GND, CON19.11, CON19.13, CON5.4, CON5.GND, CON6.4, CON6.GND, D9.C, LED1.C, LED2.C; no longer MODULE1CN8.GND@1, MODULE1CN8.GND@2
- net VDD_5V: now also CON19.9, D9.A; no longer MODULE1CN8.5V

Commit message: opencopcho is basically done
Connections:
- removed net CAN1_STBY: IC6.STBY
- removed net CAN2_STBY: IC2.STBY
- net VDD_3V3: now also CON19.7
Changed lines of the file:
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@@
 <part name="+P7" library="supply_symbols" deviceset="5V" device=""/>
 <part name="GND30" library="supply_symbols" deviceset="GND" device="" value="GND"/>
+<part name="+P6" library="supply_symbols" library_urn="urn:adsk.eagle:library:5017758" deviceset="3.3V" device=""/>
 </parts>
 <sheets>
@@
 <attribute name="VALUE" x="358.14" y="31.75" size="1.27" layer="96" font="vector" ratio="15" align="center"/>
 </instance>
-<instance part="+P7" gate="G$1" x="20.32" y="228.6" smashed="yes">
-<attribute name="VALUE" x="20.32" y="232.156" size="1.27" layer="96" font="vector" ratio="15" align="center"/>
-</instance>
-<instance part="GND30" gate="1" x="20.32" y="215.9" smashed="yes">
-<attribute name="VALUE" x="20.32" y="214.63" size="1.27" layer="96" font="vector" ratio="15" align="center"/>
+<instance part="+P7" gate="G$1" x="15.24" y="233.68" smashed="yes">
+<attribute name="VALUE" x="15.24" y="237.236" size="1.27" layer="96" font="vector" ratio="15" align="center"/>
+</instance>
+<instance part="GND30" gate="1" x="15.24" y="215.9" smashed="yes">
+<attribute name="VALUE" x="15.24" y="214.63" size="1.27" layer="96" font="vector" ratio="15" align="center"/>
+</instance>
+<instance part="+P6" gate="G$1" x="20.32" y="233.68" smashed="yes">
+<attribute name="VALUE" x="20.32" y="237.236" size="1.27" layer="96" font="vector" ratio="15" align="center"/>
 </instance>
 </instances>
@@
 <segment>
 <pinref part="CON19" gate="G$1" pin="11"/>
-<wire x1="25.4" y1="223.52" x2="20.32" y2="223.52" width="0.1524" layer="91"/>
-<wire x1="20.32" y1="223.52" x2="20.32" y2="220.98" width="0.1524" layer="91"/>
+<wire x1="25.4" y1="223.52" x2="15.24" y2="223.52" width="0.1524" layer="91"/>
+<wire x1="15.24" y1="223.52" x2="15.24" y2="220.98" width="0.1524" layer="91"/>
 <pinref part="CON19" gate="G$1" pin="13"/>
-<wire x1="20.32" y1="220.98" x2="25.4" y2="220.98" width="0.1524" layer="91"/>
+<wire x1="15.24" y1="220.98" x2="25.4" y2="220.98" width="0.1524" layer="91"/>
 <pinref part="GND30" gate="1" pin="GND"/>
-<wire x1="20.32" y1="218.44" x2="20.32" y2="220.98" width="0.1524" layer="91"/>
-<junction x="20.32" y="220.98"/>
+<wire x1="15.24" y1="218.44" x2="15.24" y2="220.98" width="0.1524" layer="91"/>
+<junction x="15.24" y="220.98"/>
 </segment>
 </net>
@@
 <segment>
 <pinref part="CON19" gate="G$1" pin="9"/>
-<wire x1="25.4" y1="226.06" x2="20.32" y2="226.06" width="0.1524" layer="91"/>
+<wire x1="25.4" y1="226.06" x2="15.24" y2="226.06" width="0.1524" layer="91"/>
 <pinref part="+P7" gate="G$1" pin="VDD_5V"/>
-<wire x1="20.32" y1="226.06" x2="20.32" y2="228.6" width="0.1524" layer="91"/>
+<wire x1="15.24" y1="226.06" x2="15.24" y2="233.68" width="0.1524" layer="91"/>
 </segment>
 </net>
@@
 <wire x1="317.5" y1="142.24" x2="317.5" y2="152.4" width="0.1524" layer="91"/>
 </segment>
-</net>
-<net name="CAN2_STBY" class="0">
-<segment>
-<pinref part="IC2" gate="G$1" pin="STBY"/>
-<wire x1="314.96" y1="149.86" x2="320.04" y2="149.86" width="0.1524" layer="91"/>
-<label x="320.04" y="149.86" size="1.27" layer="95" font="vector" xref="yes"/>
+<segment>
+<pinref part="CON19" gate="G$1" pin="7"/>
+<wire x1="25.4" y1="228.6" x2="20.32" y2="228.6" width="0.1524" layer="91"/>
+<pinref part="+P6" gate="G$1" pin="VDD_3V3"/>
+<wire x1="20.32" y1="228.6" x2="20.32" y2="233.68" width="0.1524" layer="91"/>
 </segment>
 </net>
@@
 </segment>
 </net>
-<net name="CAN1_STBY" class="0">
-<segment>
-<pinref part="IC6" gate="G$1" pin="STBY"/>
-<wire x1="314.96" y1="76.2" x2="320.04" y2="76.2" width="0.1524" layer="91"/>
-<label x="320.04" y="76.2" size="1.27" layer="95" font="vector" xref="yes"/>
-</segment>
-</net>

Commit message: basic assembly variant
Parts:
- added U$11, U$5, U$6, U$7: FIDUCIALMOUNT, usb2can_master_lib:FIDUCIALMOUNT
Other:
- moved on the sheet: CON14, CON7, R2, R40

Commit message: temporary  BOM link
Other:
- moved on the sheet: C10, C11, C12, C13, C14, C15, C16, C8, CON1, CON2, CON3, CON4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

Commit message: silk updates
Parts:
- added R11, R12: (no value), rc:R-5%-1206
- added SJ1, SJ2: (no value), usb2can_master_lib:SOLDER_JOINT
Connections:
- net CAN1_SHIELD: now also R11.1, SJ2.1
- net CAN2_SHIELD: now also R12.1, SJ1.1
- net GND: now also R11.2, R12.2, SJ1.2, SJ2.2
Changed lines of the file:
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@@
 </attributes>
 <variantdefs>
-<variantdef name="basic" current="yes"/>
+<variantdef name="basic"/>
 </variantdefs>
 <classes>
@@
 <variant name="basic" populate="no"/>
 </part>
+<part name="R11" library="rc" library_urn="urn:adsk.eagle:library:2539423" deviceset="R" device="-1206" package3d_urn="urn:adsk.eagle:package:2539464/2" technology="-5%">
+<variant name="basic" populate="no"/>
+</part>
+<part name="R12" library="rc" library_urn="urn:adsk.eagle:library:2539423" deviceset="R" device="-1206" package3d_urn="urn:adsk.eagle:package:2539464/2" technology="-5%">
+<variant name="basic" populate="no"/>
+</part>
+<part name="GND7" library="esp8266_master_lib" deviceset="GND" device=""/>
+<part name="GND31" library="esp8266_master_lib" deviceset="GND" device=""/>
+<part name="SJ1" library="usb2can_master_lib" deviceset="SOLDER_JOINT" device="">
+<variant name="basic" populate="no"/>
+</part>
+<part name="SJ2" library="usb2can_master_lib" deviceset="SOLDER_JOINT" device=""/>
 </parts>
 <sheets>
@@
 <instance part="U$6" gate="G$1" x="22.86" y="20.32" smashed="yes" rot="R270"/>
 <instance part="U$7" gate="G$1" x="22.86" y="10.16" smashed="yes" rot="R270"/>
+<instance part="R11" gate="G$1" x="238.76" y="233.68" smashed="yes" rot="R90">
+<attribute name="NAME" x="238.76" y="233.68" size="1.27" layer="95" rot="R90" align="center"/>
+<attribute name="VALUE" x="240.792" y="233.426" size="0.762" layer="96" rot="R90" align="bottom-right"/>
+<attribute name="PACKAGE" x="238.252" y="229.87" size="0.508" layer="95" rot="R90" align="center"/>
+<attribute name="TOLERANCE" x="240.792" y="233.934" size="0.762" layer="96" rot="R90"/>
+</instance>
+<instance part="R12" gate="G$1" x="236.22" y="167.64" smashed="yes" rot="R90">
+<attribute name="NAME" x="236.22" y="167.64" size="1.27" layer="95" rot="R90" align="center"/>
+<attribute name="VALUE" x="238.252" y="167.386" size="0.762" layer="96" rot="R90" align="bottom-right"/>
+<attribute name="PACKAGE" x="235.712" y="163.83" size="0.508" layer="95" rot="R90" align="center"/>
+<attribute name="TOLERANCE" x="238.252" y="167.894" size="0.762" layer="96" rot="R90"/>
+</instance>
+<instance part="GND7" gate="1" x="246.38" y="238.76" smashed="yes">
+<attribute name="VALUE" x="246.38" y="237.49" size="1.27" layer="96" font="vector" ratio="15" align="center"/>
+</instance>
+<instance part="GND31" gate="1" x="228.6" y="167.64" smashed="yes">
+<attribute name="VALUE" x="228.6" y="166.37" size="1.27" layer="96" font="vector" ratio="15" align="center"/>
+</instance>
+<instance part="SJ1" gate="G$1" x="233.68" y="167.64" smashed="yes" rot="R90">
+<attribute name="NAME" x="233.68" y="167.64" size="1.524" layer="95" font="vector" ratio="15" rot="R90" align="center"/>
+</instance>
+<instance part="SJ2" gate="G$1" x="241.3" y="233.68" smashed="yes" rot="R90">
+<attribute name="NAME" x="241.3" y="233.68" size="1.524" layer="95" font="vector" ratio="15" rot="R90" align="center"/>
+</instance>
 </instances>
 <busses>
@@
 <wire x1="15.24" y1="218.44" x2="15.24" y2="220.98" width="0.1524" layer="91"/>
 <junction x="15.24" y="220.98"/>
+</segment>
+<segment>
+<pinref part="GND7" gate="1" pin="GND"/>
+<wire x1="246.38" y1="241.3" x2="246.38" y2="243.84" width="0.1524" layer="91"/>
+<wire x1="246.38" y1="243.84" x2="243.84" y2="243.84" width="0.1524" layer="91"/>
+<wire x1="243.84" y1="243.84" x2="241.3" y2="243.84" width="0.1524" layer="91"/>
+<wire x1="241.3" y1="243.84" x2="238.76" y2="243.84" width="0.1524" layer="91"/>
+<wire x1="238.76" y1="243.84" x2="238.76" y2="241.3" width="0.1524" layer="91"/>
+<pinref part="R11" gate="G$1" pin="2"/>
+<wire x1="238.76" y1="241.3" x2="238.76" y2="238.76" width="0.1524" layer="91"/>
+<pinref part="SJ2" gate="G$1" pin="2"/>
+<wire x1="241.3" y1="238.76" x2="241.3" y2="243.84" width="0.1524" layer="91"/>
+<junction x="241.3" y="243.84"/>
+</segment>
+<segment>
+<pinref part="GND31" gate="1" pin="GND"/>
+<wire x1="228.6" y1="170.18" x2="228.6" y2="172.72" width="0.1524" layer="91"/>
+<wire x1="228.6" y1="172.72" x2="228.6" y2="175.26" width="0.1524" layer="91"/>
+<wire x1="228.6" y1="175.26" x2="233.68" y2="175.26" width="0.1524" layer="91"/>
+<pinref part="R12" gate="G$1" pin="2"/>
+<wire x1="233.68" y1="175.26" x2="236.22" y2="175.26" width="0.1524" layer="91"/>
+<wire x1="236.22" y1="175.26" x2="236.22" y2="172.72" width="0.1524" layer="91"/>
+<pinref part="SJ1" gate="G$1" pin="2"/>
+<wire x1="233.68" y1="172.72" x2="233.68" y2="175.26" width="0.1524" layer="91"/>
+<junction x="233.68" y="175.26"/>
 </segment>
 </net>
@@
 <segment>
 <pinref part="CON2" gate="G$1" pin="5"/>
-<wire x1="248.92" y1="226.06" x2="238.76" y2="226.06" width="0.1524" layer="91"/>
+<wire x1="248.92" y1="226.06" x2="241.3" y2="226.06" width="0.1524" layer="91"/>
 <label x="228.6" y="226.06" size="1.27" layer="95" rot="R180" xref="yes"/>
 <pinref part="CON1" gate="G$1" pin="5"/>
+<wire x1="241.3" y1="226.06" x2="238.76" y2="226.06" width="0.1524" layer="91"/>
 <wire x1="238.76" y1="226.06" x2="228.6" y2="226.06" width="0.1524" layer="91"/>
 <wire x1="248.92" y1="193.04" x2="238.76" y2="193.04" width="0.1524" layer="91"/>
 <wire x1="238.76" y1="193.04" x2="238.76" y2="226.06" width="0.1524" layer="91"/>
 <junction x="238.76" y="226.06"/>
+<pinref part="R11" gate="G$1" pin="1"/>
+<wire x1="238.76" y1="226.06" x2="238.76" y2="228.6" width="0.1524" layer="91"/>
+<pinref part="SJ2" gate="G$1" pin="1"/>
+<wire x1="241.3" y1="228.6" x2="241.3" y2="226.06" width="0.1524" layer="91"/>
+<junction x="241.3" y="226.06"/>
 </segment>
 <segment>
@@
 <label x="231.14" y="160.02" size="1.27" layer="95" rot="R180" xref="yes"/>
 <pinref part="CON4" gate="G$1" pin="5"/>
-<wire x1="236.22" y1="160.02" x2="231.14" y2="160.02" width="0.1524" layer="91"/>
+<wire x1="236.22" y1="160.02" x2="233.68" y2="160.02" width="0.1524" layer="91"/>
+<wire x1="233.68" y1="160.02" x2="231.14" y2="160.02" width="0.1524" layer="91"/>
 <wire x1="248.92" y1="127" x2="236.22" y2="127" width="0.1524" layer="91"/>
 <wire x1="236.22" y1="127" x2="236.22" y2="160.02" width="0.1524" layer="91"/>
 <junction x="236.22" y="160.02"/>
-</segment>
-</net>
+<pinref part="R12" gate="G$1" pin="1"/>
+<wire x1="236.22" y1="160.02" x2="236.22" y2="162.56" width="0.1524" layer="91"/>
+<pinref part="SJ1" gate="G$1" pin="1"/>
+<wire x1="233.68" y1="162.56" x2="233.68" y2="160.02" width="0.1524" layer="91"/>
+<junction x="233.68" y="160.02"/>
+</segment>
+</net>
